Commit message: first commit

File: biped/bipedal_description/urdf/bipedal.xacro (robot description, xacro)
@@ -26,10 +26,10 @@
 <link name="right_lower_femur">
   <inertial>
-    <origin xyz="0.02024419222194343 -4.543585551996729e-06 -0.006481680057536604" rpy="0 0 -0.00007"/>
+    <origin xyz="0.02024419222194343 -4.543585551996729e-06 -0.006481680057536604" rpy="0 0 0"/>
     <mass value="0.08613648212097492"/>
     <inertia ixx="5e-06" iyy="4.2e-05" izz="4.4e-05" ixy="-0.0" iyz="-0.0" ixz="-0.0"/>
   </inertial>
   <visual>
-    <origin xyz="-0.065 0.005 0.144" rpy="0 0 -0.00007"/>
+    <origin xyz="-0.065 0.005 0.144" rpy="0 0 0"/>
     <geometry>
       <mesh filename="file://$(find Bipedal_description)/meshes/right_lower_femur.stl" scale="0.001 0.001 0.001"/>
@@ -38,5 +38,5 @@
   </visual>
   <collision>
-    <origin xyz="-0.065 0.005 0.144" rpy="0 0 -0.00007"/>
+    <origin xyz="-0.065 0.005 0.144" rpy="0 0 0"/>
     <geometry>
       <mesh filename="file://$(find Bipedal_description)/meshes/right_lower_femur.stl" scale="0.001 0.001 0.001"/>
@@ -46,10 +46,10 @@
 <link name="left_lower_femur">
   <inertial>
-    <origin xyz="0.020244192221942472 -4.543585551963769e-06 -0.006481680057539546" rpy="0 0 -0.18740"/>
+    <origin xyz="0.020244192221942472 -4.543585551963769e-06 -0.006481680057539546" rpy="0 0 0"/>
     <mass value="0.08613648212097492"/>
     <inertia ixx="5e-06" iyy="4.2e-05" izz="4.4e-05" ixy="-0.0" iyz="-0.0" ixz="-0.0"/>
   </inertial>
   <visual>
-    <origin xyz="-0.065 -0.055 0.144" rpy="0 0 -0.18740"/>
+    <origin xyz="-0.065 -0.055 0.144" rpy="0 0 0"/>
     <geometry>
       <mesh filename="file://$(find Bipedal_description)/meshes/left_lower_femur.stl" scale="0.001 0.001 0.001"/>
@@ -58,5 +58,5 @@
   </visual>
   <collision>
-    <origin xyz="-0.065 -0.055 0.144" rpy="0 0 -0.18740"/>
+    <origin xyz="-0.065 -0.055 0.144" rpy="0 0 0"/>
     <geometry>
       <mesh filename="file://$(find Bipedal_description)/meshes/left_lower_femur.stl" scale="0.001 0.001 0.001"/>
@@ -66,10 +66,10 @@
 <link name="left_upper_femur">
   <inertial>
-    <origin xyz="0.02018101359279767 -0.001598133201721058 0.0064816800575395305" rpy="0 0 -0.07917"/>
+    <origin xyz="0.02018101359279767 -0.001598133201721058 0.0064816800575395305" rpy="0 0 0"/>
     <mass value="0.08613648212097492"/>
     <inertia ixx="5e-06" iyy="4.2e-05" izz="4.4e-05" ixy="3e-06" iyz="-0.0" ixz="0.0"/>
   </inertial>
   <visual>
-    <origin xyz="-0.065 -0.055 -0.004" rpy="0 0 -0.07917"/>
+    <origin xyz="-0.065 -0.055 -0.004" rpy="0 0 0"/>
     <geometry>
       <mesh filename="file://$(find Bipedal_description)/meshes/left_upper_femur.stl" scale="0.001 0.001 0.001"/>
@@ -78,5 +78,5 @@
   </visual>
   <collision>
-    <origin xyz="-0.065 -0.055 -0.004" rpy="0 0 -0.07917"/>
+    <origin xyz="-0.065 -0.055 -0.004" rpy="0 0 0"/>
     <geometry>
       <mesh filename="file://$(find Bipedal_description)/meshes/left_upper_femur.stl" scale="0.001 0.001 0.001"/>
@@ -86,10 +86,10 @@
 <link name="right_upper_femur">
   <inertial>
-    <origin xyz="0.020244192221942472 4.543585551979382e-06 0.0064816800575395305" rpy="0 0 0.17549"/>
+    <origin xyz="0.020244192221942472 4.543585551979382e-06 0.0064816800575395305" rpy="0 0 0"/>
     <mass value="0.08613648212097492"/>
     <inertia ixx="5e-06" iyy="4.2e-05" izz="4.4e-05" ixy="0.0" iyz="-0.0" ixz="0.0"/>
   </inertial>
   <visual>
-    <origin xyz="-0.065 0.005 -0.004" rpy="0 0 0.17549"/>
+    <origin xyz="-0.065 0.005 -0.004" rpy="0 0 0"/>
     <geometry>
       <mesh filename="file://$(find Bipedal_description)/meshes/right_upper_femur.stl" scale="0.001 0.001 0.001"/>
@@ -98,5 +98,5 @@
   </visual>
   <collision>
-    <origin xyz="-0.065 0.005 -0.004" rpy="0 0 0.17549"/>
+    <origin xyz="-0.065 0.005 -0.004" rpy="0 0 0"/>
     <geometry>
       <mesh filename="file://$(find Bipedal_description)/meshes/right_upper_femur.stl" scale="0.001 0.001 0.001"/>
@@ -225,5 +225,5 @@
 </link>
 <joint name="right_lower_hip_joint" type="revolute">
-  <origin xyz="0.065 -0.005 -0.144" rpy="0 0 00 0 0.00007/>
+  <origin xyz="0.065 -0.005 -0.144" rpy="0 0 0"/>
   <parent link="base_link"/>
   <child link="right_lower_femur"/>
@@ -232,5 +232,5 @@
 </joint>
 <joint name="left_lower_hip_joint" type="revolute">
-  <origin xyz="0.065 0.055 -0.144" rpy="0 0 00 0 0.18740/>
+  <origin xyz="0.065 0.055 -0.144" rpy="0 0 0.18737"/>
   <parent link="base_link"/>
   <child link="left_lower_femur"/>
@@ -239,5 +239,5 @@
 </joint>
 <joint name="left_upper_hip_joint" type="revolute">
-  <origin xyz="0.065 0.055 0.004" rpy="0 0 -0.087266"/>
+  <origin xyz="0.065 0.055 0.004" rpy="0 0 0.07917"/>
   <parent link="base_link"/>
   <child link="left_upper_femur"/>
@@ -246,5 +246,5 @@
 </joint>
 <joint name="right_upper_hip_joint" type="revolute">
-  <origin xyz="0.065 -0.005 0.004" rpy="0 0 00 0 0.07917/>
+  <origin xyz="0.065 -0.005 0.004" rpy="0 0 -0.17552"/>
   <parent link="base_link"/>
   <child link="right_upper_femur"/>
@@ -253,5 +253,5 @@
 </joint>
 <joint name="left_knee_joint" type="revolute">
-  <origin xyz="0.055000 0.0 0.004" rpy="0 0 00 0 -0.17549/>
+  <origin xyz="0.054828 -0.00435 0.004" rpy="0 0 0"/>
   <parent link="left_upper_femur"/>
   <child link="left_tibia"/>
@@ -260,5 +260,5 @@
 </joint>
 <joint name="right_knee_joint" type="revolute">
-  <origin xyz="0.055000 0.0 -0.004" rpy="0 0 00 0 -0.00000/>
+  <origin xyz="0.055 -4e-06 -0.004" rpy="0 0 0"/>
   <parent link="right_lower_femur"/>
   <child link="right_tibia"/>
@@ -267,5 +267,5 @@
 </joint>
 <joint name="right_upper_knee_to_linkage1" type="revolute">
-  <origin xyz="0.161226 0.0 0.004" rpy="0 0 00 0 -0.00000/>
+  <origin xyz="0.15875 0.028148 0.004" rpy="0 0 0"/>
   <parent link="right_upper_femur"/>
   <child link="inner_linkage_1"/>
@@ -274,5 +274,5 @@
 </joint>
 <joint name="left_lower_knee_to_linkage2" type="revolute">
-  <origin xyz="0.161049 0.0 -0.004" rpy="0 0 00 0 -0.00000/>
+  <origin xyz="0.158229 -0.030004 -0.004" rpy="0 0 0"/>
   <parent link="left_lower_femur"/>
   <child link="inner_linkage_2"/>
@@ -281,5 +281,5 @@
 </joint>
 <joint name="right_tibia_to_linkage2" type="revolute">
-  <origin xyz="0.103229 0.03 0.0" rpy="0 0 00 0 -0.00000/>
+  <origin xyz="0.103229 0.03 0.0" rpy="0 0 0"/>
   <parent link="right_tibia"/>
   <child link="inner_linkage_2"/>
