Commit message: updated knee joint but the tibia's joint issue

File: biped/bipedal_URDF/assembly_description/urdf/assembly.xacro (robot description, xacro)
@@ -1,296 +1,297 @@
 <?xml version="1.0" ?>
+<!--
+  Bipedal robot - 5-bar parallel closed-loop legs.
+  ============================================================================
+  MECHANISM
+  ============================================================================
+  Each leg is a planar 5-bar linkage (2 DOF) lying in the sagittal plane:
+        pelvis
+      H_rear o========= 60 mm ========o H_front     [ground link = base_link]
+              \                      /
+               \ 55 mm        55 mm /               [the two femurs]
+                \                  /
+          K_rear o                o K_front         [the two knees]
+                  \              /
+           107.5   \            /   107.5 mm        [the two shanks]
+                    \          /
+                     \        /
+                      o======o
+                       FOOT                         [loop-closure pivot]
+  Both hips are actuated; both knees are PASSIVE and fully determined by the
+  hip angles through the loop-closure constraint. Link lengths were measured
+  directly off the CAD meshes and the loop closes to within 1 micron at the
+  CAD zero pose.
+  ============================================================================
+  WHY THERE IS NO <joint> FOR THE FOOT PIVOT
+  ============================================================================
+  URDF can only describe a kinematic TREE. A 5-bar has one independent loop
+  per leg, so exactly one joint per leg must be left out of the tree - here
+  that is the foot pivot, "<side>_foot_closure". Each leg therefore contributes
+  4 tree joints (2 hips + 2 knees) and 1 cut joint.
+  The cut is NOT a modelling error and must NOT be "fixed" by giving the
+  inner linkage a second parent (a link with two parents is invalid URDF and
+  is what caused the earlier model to load with dangling, disconnected knees).
+  To make the linkage render CLOSED in RViz, run the five_bar_state_publisher
+  node shipped with this package: it takes the 2 hip angles per leg, solves
+  the closure analytically, and publishes all 8 joint values consistently.
+  See launch/display.launch.py.
+  For Gazebo, the real revolute constraint is re-attached in assembly.gazebo.
+  ============================================================================
+  FRAMES
+  ============================================================================
+  The CAD was exported with +X pointing DOWN and +Z pointing across the hips.
+  base_footprint re-expresses that in the ROS convention (REP-103: X forward,
+  Y left, Z up) via a single fixed joint, so the robot stands upright in RViz
+  with its feet on the grid. All link/joint numbers below are kept in the
+  original CAD frame so they can be checked against the Fusion export.
+  Zero configuration == the CAD assembly pose.
+-->
 <robot name="assembly" xmlns:xacro="http://www.ros.org/wiki/xacro">
-<xacro:include filename="$(find assembly_description)/urdf/materials.xacro" />
-<xacro:include filename="$(find assembly_description)/urdf/assembly.trans" />
-<xacro:include filename="$(find assembly_description)/urdf/assembly.gazebo" />
-<link name="base_link">
-  <inertial>
-    <origin xyz="0.021483404329702544 0.02602124280867646 -0.06951546728903525" rpy="0 0 0"/>
-    <mass value="5.554037091220957"/>
-    <inertia ixx="0.019731" iyy="0.024901" izz="0.017821" ixy="0.000405" iyz="-2.5e-05" ixz="0.00012"/>
-  </inertial>
-  <visual>
-    <origin xyz="0 0 0" rpy="0 0 0"/>
-    <geometry>
-      <mesh filename="file://$(find assembly_description)/meshes/base_link.stl" scale="0.001 0.001 0.001"/>
-    </geometry>
-    <material name="silver"/>
-  </visual>
-  <collision>
-    <origin xyz="0 0 0" rpy="0 0 0"/>
-    <geometry>
-      <mesh filename="file://$(find assembly_description)/meshes/base_link.stl" scale="0.001 0.001 0.001"/>
-    </geometry>
-  </collision>
-</link>
-<link name="Combined_femur_1">
-  <inertial>
-    <origin xyz="0.020244192221942445 -4.543585551996729e-06 -0.006481680057539518" rpy="0 0 0"/>
-    <mass value="0.08613648212097492"/>
-    <inertia ixx="5e-06" iyy="4.2e-05" izz="4.4e-05" ixy="-0.0" iyz="-0.0" ixz="-0.0"/>
-  </inertial>
-  <visual>
-    <origin xyz="-0.065 0.005 0.144" rpy="0 0 0"/>
-    <geometry>
-      <mesh filename="file://$(find assembly_description)/meshes/Combined_femur_1.stl" scale="0.001 0.001 0.001"/>
-    </geometry>
-    <material name="silver"/>
-  </visual>
-  <collision>
-    <origin xyz="-0.065 0.005 0.144" rpy="0 0 0"/>
-    <geometry>
-      <mesh filename="file://$(find assembly_description)/meshes/Combined_femur_1.stl" scale="0.001 0.001 0.001"/>
-    </geometry>
-  </collision>
-</link>
-<link name="Combined_femur__3__1">
-  <inertial>
-    <origin xyz="0.020244192221942472 -4.543585552012341e-06 -0.006481680057539518" rpy="0 0 0"/>
-    <mass value="0.08613648212097492"/>
-    <inertia ixx="5e-06" iyy="4.2e-05" izz="4.4e-05" ixy="-0.0" iyz="-0.0" ixz="-0.0"/>
-  </inertial>
-  <visual>
-    <origin xyz="-0.065 -0.055 0.144" rpy="0 0 0"/>
-    <geometry>
-      <mesh filename="file://$(find assembly_description)/meshes/Combined_femur__3__1.stl" scale="0.001 0.001 0.001"/>
-    </geometry>
-    <material name="silver"/>
-  </visual>
-  <collision>
-    <origin xyz="-0.065 -0.055 0.144" rpy="0 0 0"/>
-    <geometry>
-      <mesh filename="file://$(find assembly_description)/meshes/Combined_femur__3__1.stl" scale="0.001 0.001 0.001"/>
-    </geometry>
-  </collision>
-</link>
-<link name="Combined_femur__1__1">
-  <inertial>
-    <origin xyz="0.0202441922219425 4.543585551963769e-06 0.0064816800575395305" rpy="0 0 0"/>
-    <mass value="0.08613648212097492"/>
-    <inertia ixx="5e-06" iyy="4.2e-05" izz="4.4e-05" ixy="0.0" iyz="-0.0" ixz="0.0"/>
-  </inertial>
-  <visual>
-    <origin xyz="-0.065 -0.055 -0.004" rpy="0 0 0"/>
-    <geometry>
-      <mesh filename="file://$(find assembly_description)/meshes/Combined_femur__1__1.stl" scale="0.001 0.001 0.001"/>
-    </geometry>
-    <material name="silver"/>
-  </visual>
-  <collision>
-    <origin xyz="-0.065 -0.055 -0.004" rpy="0 0 0"/>
-    <geometry>
-      <mesh filename="file://$(find assembly_description)/meshes/Combined_femur__1__1.stl" scale="0.001 0.001 0.001"/>
-    </geometry>
-  </collision>
-</link>
-<link name="Combined_femur__2__1">
-  <inertial>
-    <origin xyz="0.0202441922219425 4.543585551957698e-06 0.006481680057539529" rpy="0 0 0"/>
-    <mass value="0.08613648212097492"/>
-    <inertia ixx="5e-06" iyy="4.2e-05" izz="4.4e-05" ixy="0.0" iyz="-0.0" ixz="0.0"/>
-  </inertial>
-  <visual>
-    <origin xyz="-0.065 0.005 -0.004" rpy="0 0 0"/>
-    <geometry>
-      <mesh filename="file://$(find assembly_description)/meshes/Combined_femur__2__1.stl" scale="0.001 0.001 0.001"/>
-    </geometry>
-    <material name="silver"/>
-  </visual>
-  <collision>
-    <origin xyz="-0.065 0.005 -0.004" rpy="0 0 0"/>
-    <geometry>
-      <mesh filename="file://$(find assembly_description)/meshes/Combined_femur__2__1.stl" scale="0.001 0.001 0.001"/>
-    </geometry>
-  </collision>
-</link>
-<link name="combined_motor_tibia__1__1">
-  <inertial>
-    <origin xyz="0.0916133412345842 -0.026627976073639873 -0.007967217020517796" rpy="0 0 0"/>
-    <mass value="0.5702684639688947"/>
-    <inertia ixx="0.000219" iyy="0.000581" izz="0.000555" ixy="0.000115" iyz="-2e-05" ixz="6.6e-05"/>
-  </inertial>
-  <visual>
-    <origin xyz="-0.12 -0.055004 -0.008" rpy="0 0 0"/>
-    <geometry>
-      <mesh filename="file://$(find assembly_description)/meshes/combined_motor_tibia__1__1.stl" scale="0.001 0.001 0.001"/>
-    </geometry>
-    <material name="silver"/>
-  </visual>
-  <collision>
-    <origin xyz="-0.12 -0.055004 -0.008" rpy="0 0 0"/>
-    <geometry>
-      <mesh filename="file://$(find assembly_description)/meshes/combined_motor_tibia__1__1.stl" scale="0.001 0.001 0.001"/>
-    </geometry>
-  </collision>
-</link>
-<link name="combined_motor_tibia_1">
-  <inertial>
-    <origin xyz="0.09161334123458417 0.026627976073640078 0.00796721702051778" rpy="0 0 0"/>
-    <mass value="0.5702684639688947"/>
-    <inertia ixx="0.000219" iyy="0.000581" izz="0.000555" ixy="-0.000115" iyz="-2e-05" ixz="-6.6e-05"/>
-  </inertial>
-  <visual>
-    <origin xyz="-0.12 0.005004 0.148" rpy="0 0 0"/>
-    <geometry>
-      <mesh filename="file://$(find assembly_description)/meshes/combined_motor_tibia_1.stl" scale="0.001 0.001 0.001"/>
-    </geometry>
-    <material name="silver"/>
-  </visual>
-  <collision>
-    <origin xyz="-0.12 0.005004 0.148" rpy="0 0 0"/>
-    <geometry>
-      <mesh filename="file://$(find assembly_description)/meshes/combined_motor_tibia_1.stl" scale="0.001 0.001 0.001"/>
-    </geometry>
-  </collision>
-</link>
-<link name="leg2_knee_tibia_1">
-  <inertial>
-    <origin xyz="0.060273696368209784 0.017517055517382807 -0.001667704624892007" rpy="0 0 0"/>
-    <mass value="0.16915049183932718"/>
-    <inertia ixx="4.6e-05" iyy="0.000236" izz="0.00028" ixy="-6e-05" iyz="3e-06" ixz="1.1e-05"/>
-  </inertial>
-  <visual>
-    <origin xyz="-0.12 0.004996 -0.008" rpy="0 0 0"/>
-    <geometry>
-      <mesh filename="file://$(find assembly_description)/meshes/tibia_2__1__1.stl" scale="0.001 0.001 0.001"/>
-    </geometry>
-    <material name="silver"/>
-  </visual>
-  <collision>
-    <origin xyz="-0.12 0.004996 -0.008" rpy="0 0 0"/>
-    <geometry>
-      <mesh filename="file://$(find assembly_description)/meshes/tibia_2__1__1.stl" scale="0.001 0.001 0.001"/>
-    </geometry>
-  </collision>
-</link>
-<link name="leg1_knee_tibia_1">
-  <inertial>
-    <origin xyz="0.060273696368209784 -0.017517055517382668 0.001667704624891908" rpy="0 0 0"/>
-    <mass value="0.16915049183932718"/>
-    <inertia ixx="4.6e-05" iyy="0.000236" izz="0.00028" ixy="6e-05" iyz="3e-06" ixz="-1.1e-05"/>
-  </inertial>
-  <visual>
-    <origin xyz="-0.12 -0.054996 0.148" rpy="0 0 0"/>
-    <geometry>
-      <mesh filename="file://$(find assembly_description)/meshes/tibia_2_1.stl" scale="0.001 0.001 0.001"/>
-    </geometry>
-    <material name="silver"/>
-  </visual>
-  <collision>
-    <origin xyz="-0.12 -0.054996 0.148" rpy="0 0 0"/>
-    <geometry>
-      <mesh filename="file://$(find assembly_description)/meshes/tibia_2_1.stl" scale="0.001 0.001 0.001"/>
-    </geometry>
-  </collision>
-</link>
-<link name="leg1_knee_tibia_2">
-  <inertial>
-    <origin xyz="-0.04295530363179023 0.012482944482617334 0.001667704624891908" rpy="0 0 0"/>
-    <mass value="0.16915049183932718"/>
-    <inertia ixx="4.6e-05" iyy="0.000236" izz="0.00028" ixy="6e-05" iyz="3e-06" ixz="-1.1e-05"/>
-  </inertial>
-  <visual>
-    <origin xyz="-0.223229 -0.024996 0.148" rpy="0 0 0"/>
-    <geometry>
-      <mesh filename="file://$(find assembly_description)/meshes/tibia_2_1.stl" scale="0.001 0.001 0.001"/>
-    </geometry>
-    <material name="silver"/>
-  </visual>
-  <collision>
-    <origin xyz="-0.223229 -0.024996 0.148" rpy="0 0 0"/>
-    <geometry>
-      <mesh filename="file://$(find assembly_description)/meshes/tibia_2_1.stl" scale="0.001 0.001 0.001"/>
-    </geometry>
-  </collision>
-</link>
-<link name="leg2_knee_tibia_2">
-  <inertial>
-    <origin xyz="-0.04295530363179023 -0.012482944482617192 -0.001667704624892007" rpy="0 0 0"/>
-    <mass value="0.16915049183932718"/>
-    <inertia ixx="4.6e-05" iyy="0.000236" izz="0.00028" ixy="-6e-05" iyz="3e-06" ixz="1.1e-05"/>
-  </inertial>
-  <visual>
-    <origin xyz="-0.223229 -0.025004 -0.008" rpy="0 0 0"/>
-    <geometry>
-      <mesh filename="file://$(find assembly_description)/meshes/tibia_2__1__1.stl" scale="0.001 0.001 0.001"/>
-    </geometry>
-    <material name="silver"/>
-  </visual>
-  <collision>
-    <origin xyz="-0.223229 -0.025004 -0.008" rpy="0 0 0"/>
-    <geometry>
-      <mesh filename="file://$(find assembly_description)/meshes/tibia_2__1__1.stl" scale="0.001 0.001 0.001"/>
-    </geometry>
-  </collision>
-</link>
-<joint name="Revolute 1" type="revolute">
-  <origin xyz="0.065 -0.005 -0.144" rpy="0 0 0"/>
-  <parent link="base_link"/>
-  <child link="Combined_femur_1"/>
-  <axis xyz="0.0 0.0 1.0"/>
-  <limit upper="-2.094395" lower="-4.18879" effort="100" velocity="100"/>
-</joint>
-<joint name="Revolute 2" type="revolute">
-  <origin xyz="0.065 0.055 -0.144" rpy="0 0 0"/>
-  <parent link="base_link"/>
-  <child link="Combined_femur__3__1"/>
-  <axis xyz="0.0 0.0 1.0"/>
-  <limit upper="-2.094395" lower="-4.18879" effort="100" velocity="100"/>
-</joint>
-<joint name="Revolute 3" type="revolute">
-  <origin xyz="0.065 0.055 0.004" rpy="0 0 0"/>
-  <parent link="base_link"/>
-  <child link="Combined_femur__1__1"/>
-  <axis xyz="0.0 0.0 -1.0"/>
-  <limit upper="-2.094395" lower="-4.18879" effort="100" velocity="100"/>
-</joint>
-<joint name="Revolute 4" type="revolute">
-  <origin xyz="0.065 -0.005 0.004" rpy="0 0 0"/>
-  <parent link="base_link"/>
-  <child link="Combined_femur__2__1"/>
-  <axis xyz="0.0 0.0 -1.0"/>
-  <limit upper="-2.094395" lower="-4.18879" effort="100" velocity="100"/>
-</joint>
-<joint name="Revolute 5" type="revolute">
-  <origin xyz="0.055 4e-06 0.004" rpy="0 0 0"/>
-  <parent link="Combined_femur__1__1"/>
-  <child link="combined_motor_tibia__1__1"/>
-  <axis xyz="-0.0 -0.0 -1.0"/>
-  <limit upper="3.926991" lower="-0.785398" effort="100" velocity="100"/>
-</joint>
-<joint name="Revolute 6" type="revolute">
-  <origin xyz="0.055 -4e-06 -0.004" rpy="0 0 0"/>
-  <parent link="Combined_femur_1"/>
-  <child link="combined_motor_tibia_1"/>
-  <axis xyz="0.0 0.0 1.0"/>
-  <limit upper="3.926991" lower="-0.785398" effort="100" velocity="100"/>
-</joint>
-<joint name="Revolute 7" type="revolute">
-  <origin xyz="0.158229 0.030004 0.004" rpy="0 0 0"/>
-  <parent link="Combined_femur__2__1"/>
-  <child link="leg2_knee_tibia_1"/>
-  <axis xyz="-0.0 0.0 -1.0"/>
-  <limit upper="3.926991" lower="-0.785398" effort="100" velocity="100"/>
-</joint>
-<joint name="Revolute 8" type="revolute">
-  <origin xyz="0.158229 -0.030004 -0.004" rpy="0 0 0"/>
-  <parent link="Combined_femur__3__1"/>
-  <child link="leg1_knee_tibia_1"/>
-  <axis xyz="0.0 0.0 1.0"/>
-  <limit upper="3.926991" lower="-0.785398" effort="100" velocity="100"/>
-</joint>
-<joint name="Revolute 9" type="revolute">
-  <origin xyz="0.103229 0.03 0.0" rpy="0 0 0"/>
-  <parent link="combined_motor_tibia_1"/>
-  <child link="leg1_knee_tibia_2"/>
-  <axis xyz="-0.0 0.0 -1.0"/>
-  <limit upper="-3.403392" lower="-5.759587" effort="100" velocity="100"/>
-</joint>
-<joint name="Revolute 10" type="revolute">
-  <origin xyz="0.103229 -0.03 0.0" rpy="0 0 0"/>
-  <parent link="combined_motor_tibia__1__1"/>
-  <child link="leg2_knee_tibia_2"/>
-  <axis xyz="0.0 0.0 1.0"/>
-  <limit upper="2.96706" lower="0.523599" effort="100" velocity="100"/>
-</joint>
+  <xacro:include filename="$(find assembly_description)/urdf/materials.xacro" />
+  <xacro:include filename="$(find assembly_description)/urdf/assembly.trans" />
+  <xacro:include filename="$(find assembly_description)/urdf/assembly.gazebo" />
+  <!-- ===================================================================== -->
+  <!-- Measured mechanism parameters (metres)                                -->
+  <!-- ===================================================================== -->
+  <xacro:property name="femur_len"   value="0.055"   />
+  <xacro:property name="shank_len"   value="0.1075"  />
+  <xacro:property name="hip_spacing" value="0.060"   />
+  <!-- lowest point of the foot meshes at the zero pose, in CAD +X -->
+  <xacro:property name="stand_height" value="0.2018" />
+  <!-- The CAD origin is not centred between the legs (they sit at CAD
+       z = +0.008 and -0.148, and the feet at CAD y = +0.0146), so the model
+       would otherwise render hanging off to one side of the grid. These two
+       offsets put base_footprint midway between the feet. -->
+  <xacro:property name="centre_x" value="-0.0146" />
+  <xacro:property name="centre_y" value="-0.0700" />
+  <!-- Actuated hip travel about the CAD pose. Verified by sweeping the
+       closure solver: over +-60 deg the mechanism stays 45 mm away from the
+       stretched singularity and every pose is reachable. Going to +-90 deg
+       folds the linkage back through itself, so do not widen this without
+       re-checking self-collision. -->
+  <xacro:property name="hip_lower"  value="-1.047198" />  <!-- -60 deg -->
+  <xacro:property name="hip_upper"  value="1.047198"  />  <!-- +60 deg -->
+  <!-- Passive knee travel: the range the dependent knees actually sweep over
+       the hip workspace above, plus a small margin. -->
+  <xacro:property name="knee_rear_lower"  value="-1.522119" />
+  <xacro:property name="knee_rear_upper"  value="1.189686"  />
+  <xacro:property name="knee_front_lower" value="-1.199474" />
+  <xacro:property name="knee_front_upper" value="1.756498"  />
+  <xacro:property name="joint_effort"   value="100" />
+  <xacro:property name="joint_velocity" value="100" />
+  <xacro:property name="joint_damping"  value="0.05" />
+  <!-- ===================================================================== -->
+  <!-- Helper macros                                                         -->
+  <!-- ===================================================================== -->
+  <!-- A CAD-exported body: the mesh lives in assembly coordinates, so the
+       visual origin is simply minus the link-frame position. -->
+  <xacro:macro name="cad_link" params="name mesh colour mass ixx iyy izz ixy iyz ixz
+                                       com_x com_y com_z org_x org_y org_z">
+    <link name="${name}">
+      <inertial>
+        <origin xyz="${com_x} ${com_y} ${com_z}" rpy="0 0 0"/>
+        <mass value="${mass}"/>
+        <inertia ixx="${ixx}" iyy="${iyy}" izz="${izz}"
+                 ixy="${ixy}" iyz="${iyz}" ixz="${ixz}"/>
+      </inertial>
+      <visual>
+        <origin xyz="${-org_x} ${-org_y} ${-org_z}" rpy="0 0 0"/>
+        <geometry>
+          <mesh filename="file://$(find assembly_description)/meshes/${mesh}"
+                scale="0.001 0.001 0.001"/>
+        </geometry>
+        <material name="${colour}"/>
+      </visual>
+      <collision>
+        <origin xyz="${-org_x} ${-org_y} ${-org_z}" rpy="0 0 0"/>
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
File: biped/bipedal_URDF/assembly_description/urdf/assembly_view.urdf (robot description, URDF)
Before this commit: robot assembly, 12 links, 11 joints
Links:
- link base_link: geometry collision mesh filename=../meshes/pelvis.stl scale=0.001 0.001 0.001; visual mesh filename=../meshes/pelvis.stl scale=0.001 0.001 0.001
- link left_femur_front: geometry collision mesh filename=../meshes/left_femur_front.stl scale=0.001 0.001 0.001; visual mesh filename=../meshes/left_femur_front.stl scale=0.001 0.001 0.001
- link left_femur_rear: geometry collision mesh filename=../meshes/left_femur_rear.stl scale=0.001 0.001 0.001; visual mesh filename=../meshes/left_femur_rear.stl scale=0.001 0.001 0.001
- link left_shank_front: geometry collision mesh filename=../meshes/left_shank_front.stl scale=0.001 0.001 0.001; visual mesh filename=../meshes/left_shank_front.stl scale=0.001 0.001 0.001
- link left_shank_rear: geometry collision mesh filename=../meshes/left_shank_rear.stl scale=0.001 0.001 0.001; visual mesh filename=../meshes/left_shank_rear.stl scale=0.001 0.001 0.001
- link right_femur_front: geometry collision mesh filename=../meshes/right_femur_front.stl scale=0.001 0.001 0.001; visual mesh filename=../meshes/right_femur_front.stl scale=0.001 0.001 0.001
- link right_femur_rear: geometry collision mesh filename=../meshes/right_femur_rear.stl scale=0.001 0.001 0.001; visual mesh filename=../meshes/right_femur_rear.stl scale=0.001 0.001 0.001
- link right_shank_front: geometry collision mesh filename=../meshes/right_shank_front.stl scale=0.001 0.001 0.001; visual mesh filename=../meshes/right_shank_front.stl scale=0.001 0.001 0.001
- link right_shank_rear: geometry collision mesh filename=../meshes/right_shank_rear.stl scale=0.001 0.001 0.001; visual mesh filename=../meshes/right_shank_rear.stl scale=0.001 0.001 0.001

File: biped/bipedal_URDF/assembly_description/urdf/materials.xacro (robot description, xacro)
@@ -1,6 +1,23 @@
 <?xml version="1.0" ?>
-<robot name="assembly" xmlns:xacro="http://www.ros.org/wiki/xacro" >
-<material name="silver">
-  <color rgba="0.700 0.700 0.700 1.000"/>
-</material>
+<!-- Distinct colours per role so the parallel linkage is readable in RViz:
+     the two shanks of a leg are deliberately different colours, which makes
+     it immediately obvious whether the loop is closing at the foot. -->
+<robot name="assembly" xmlns:xacro="http://www.ros.org/wiki/xacro">
+  <material name="pelvis_grey">
+    <color rgba="0.45 0.47 0.50 1.0"/>
+  </material>
+  <material name="femur_orange">
+    <color rgba="0.95 0.55 0.15 1.0"/>
+  </material>
+  <!-- motor-carrying shank -->
+  <material name="shank_dark">
+    <color rgba="0.18 0.20 0.23 1.0"/>
+  </material>
+  <!-- thin inner linkage bar -->
+  <material name="linkage_blue">
+    <color rgba="0.20 0.50 0.85 1.0"/>
+  </material>
+  <material name="silver">
+    <color rgba="0.700 0.700 0.700 1.000"/>
+  </material>
 </robot>
